File: SPRO3 - PCB/SPRO3 - PCB.kicad_sch (KiCad schematic)
At the start: 39 parts

Commit message: Added footnotes to the main PCB and tested and tested stuff in the board editor
Parts:
- C1, C10, C11, C2, C3, C5, C6, C7, C8, C9: renamed from C?; footprint (none) -> Capacitor_THT:CP_Radial_D5.0mm_P2.50mm
- C4: renamed from C?; footprint (none) -> Capacitor_THT:C_Disc_D3.8mm_W2.6mm_P2.50mm
- D1: renamed from D?; footprint (none) -> Diode_THT:D_DO-41_SOD81_P10.16mm_Horizontal
- D2: renamed from D?; footprint (none) -> LED_THT:LED_D5.0mm
- J1: renamed from J?; value 2nd PCB -> Power Input; footprint (none) -> TerminalBlock:TerminalBlock_bornier-2_P5.08mm
- J10, J11, J12, J13, J14, J15, J3, J5, J8, J9: renamed from J?; footprint (none) -> Connector_PinHeader_2.54mm:PinHeader_1x03_P2.54mm_Vertical
- J16, J6: renamed from J?; footprint (none) -> Connector_PinHeader_2.54mm:PinHeader_1x04_P2.54mm_Vertical
- J2: renamed from J?; footprint (none) -> Connector_PinHeader_2.54mm:PinHeader_1x02_P2.54mm_Vertical
- J4: renamed from J?; footprint (none) -> Connector_PinHeader_2.54mm:PinHeader_1x06_P2.54mm_Vertical
- J7: renamed from J?; footprint (none) -> Connector_PinSocket_2.54mm:PinSocket_1x04_P2.54mm_Vertical
- R1, R2, R3, R4, R5: renamed from R?; footprint (none) -> Resistor_THT:R_Axial_DIN0207_L6.3mm_D2.5mm_P10.16mm_Horizontal
- SW1: renamed from SW?; footprint (none) -> Connector_Wire:SolderWire-0.75sqmm_1x03_P4.8mm_D1.25mm_OD2.3mm
- TH1: renamed from TH?; footprint (none) -> Resistor_THT:R_Axial_DIN0204_L3.6mm_D1.6mm_P2.54mm_Vertical
- U1: renamed from U?; footprint (none) -> Package_DIP:DIP-8_W7.62mm
- U2: renamed from U?; footprint (none) -> Package_DIP:DIP-16_W7.62mm
- gave numbers to parts that had none: 1
Connections:
- net PC0 is gone; now on net IN1: J4.2 (Pin_2)
- net PC1 is gone; now on net IN2: J4.3 (Pin_3)
- net PC2 is gone; now on net IN3: J4.4 (Pin_4)
- net PC3 is gone; now on net IN4: J4.5 (Pin_5)
- net +5V: now also J10.2 (Pin_2), J11.2 (Pin_2), J12.2 (Pin_2), J13.2 (Pin_2), J14.2 (Pin_2), J15.2 (Pin_2), J8.2 (Pin_2), J9.2 (Pin_2); no longer J10.1 (Pin_1), J11.1 (Pin_1), J12.1 (Pin_1), J13.1 (Pin_1), J14.1 (Pin_1), J15.1 (Pin_1), J8.1 (Pin_1), J9.1 (Pin_1)
- net A: now also A1.12 (D9); no longer A1.13 (D10)
- net B: now also A1.13 (D10); no longer A1.12 (D9)
- net IN1: now also A1.16 (D13); no longer A1.19 (A0)
- net IN2: now also A1.19 (A0); no longer A1.20 (A1)
- net IN3: now also A1.20 (A1); no longer A1.21 (A2)
- net IN4: now also A1.21 (A2); no longer A1.16 (D13)
- net at U2.4 (X7): now also J15.1 (Pin_1); no longer J15.2 (Pin_2)
- net at U2.5 (X5): now also J13.1 (Pin_1); no longer J13.2 (Pin_2)
- net at U2.14 (X1): now also J9.1 (Pin_1); no longer J9.2 (Pin_2)
- net at U2.1 (X4): now also J12.1 (Pin_1); no longer J12.2 (Pin_2)
- net at U2.12 (X3): now also J11.1 (Pin_1); no longer J11.2 (Pin_2)
- net at U2.13 (X0): now also J8.1 (Pin_1); no longer J8.2 (Pin_2)
- net at U2.15 (X2): now also J10.1 (Pin_1); no longer J10.2 (Pin_2)
- net at U2.2 (X6): now also J14.1 (Pin_1); no longer J14.2 (Pin_2)
- no-connect marks 4 -> 16
Other:
- moved on the sheet: C10, D2

Commit message: First attempt at designing the main PCB board
Connections:
- net IN1: now also J4.3 (Pin_3); no longer J4.2 (Pin_2)
- net IN2: now also A1.22 (A3), J4.6 (Pin_6); no longer A1.19 (A0), J4.3 (Pin_3)
- net NTC_Vout(ADC3): now also A1.19 (A0); no longer A1.22 (A3)
- net OC0B: now also J4.2 (Pin_2); no longer J4.6 (Pin_6)
Changed lines of the file:
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@@
+		)
+	)
+	(text "IN3"
+		(exclude_from_sim no)
+		(at 144.78 170.434 0)
+		(effects
+			(font
+				(size 1.27 1.27)
+			)
+		)
+	)
+	(text "Thermistor"
+		(exclude_from_sim no)
+		(at 59.182 186.436 0)
+		(effects
+			(font
+				(size 2.5 2.5)
+			)
+		)
+	)
+	(text "Power Input"
+		(exclude_from_sim no)
+		(at 57.15 80.772 0)
+		(effects
+			(font
+				(size 2.5 2.5)
+			)
+		)
+	)
+	(text "Ultrasonic Sensors"
+		(exclude_from_sim no)
+		(at 226.314 113.538 0)
+		(effects
+			(font
+				(size 2.5 2.5)
+			)
+		)
+	)
+	(text "VCC"
+		(exclude_from_sim no)
+		(at 40.386 40.894 0)
+		(effects
+			(font
+				(size 1.27 1.27)
+			)
 		)
 	)
 	(text "IN2"
 		(exclude_from_sim no)
-		(at 144.78 170.434 0)
-		(effects
-			(font
-				(size 1.27 1.27)
-			)
-		)
-	)
-	(text "Thermistor"
-		(exclude_from_sim no)
-		(at 59.182 186.436 0)
-		(effects
-			(font
-				(size 2.5 2.5)
-			)
-		)
-	)
-	(text "Power Input"
-		(exclude_from_sim no)
-		(at 57.15 80.772 0)
-		(effects
-			(font
-				(size 2.5 2.5)
-			)
-		)
-	)
-	(text "Ultrasonic Sensors"
-		(exclude_from_sim no)
-		(at 226.314 113.538 0)
-		(effects
-			(font
-				(size 2.5 2.5)
-			)
-		)
-	)
-	(text "VCC"
-		(exclude_from_sim no)
-		(at 40.386 40.894 0)
+		(at 144.78 165.354 0)
+		(effects
+			(font
+				(size 1.27 1.27)
+			)
+		)
+	)
+	(text "H Bridge Module"
+		(exclude_from_sim no)
+		(at 139.954 185.928 0)
+		(effects
+			(font
+				(size 2.5 2.5)
+			)
+		)
+	)
+	(text "GND"
+		(exclude_from_sim no)
+		(at 120.65 132.334 0)
 		(effects
 			(font
@@
 	)
 	(text "IN4"
-		(exclude_from_sim no)
-		(at 144.78 165.354 0)
-		(effects
-			(font
-				(size 1.27 1.27)
-			)
-		)
-	)
-	(text "H Bridge Module"
-		(exclude_from_sim no)
-		(at 139.954 185.928 0)
-		(effects
-			(font
-				(size 2.5 2.5)
-			)
-		)
-	)
-	(text "GND"
-		(exclude_from_sim no)
-		(at 120.65 132.334 0)
-		(effects
-			(font
-				(size 1.27 1.27)
-			)
-		)
-	)
-	(text "IN3"
 		(exclude_from_sim no)
 		(at 144.78 167.894 0)
@@
 		)
 	)
-	(label "OC0B"
+	(label "IN2"
 		(at 134.62 162.56 180)
 		(fields_autoplaced yes)
@@
 		)
 	)
-	(label "NTC_Vout(ADC3)"
+	(label "IN2"
 		(at 148.59 62.23 0)
 		(fields_autoplaced yes)
@@
 		)
 	)
-	(label "IN1"
+	(label "OC0B"
 		(at 134.62 172.72 180)
 		(fields_autoplaced yes)
@@
 		)
 	)
-	(label "IN2"
+	(label "IN1"
 		(at 134.62 170.18 180)
 		(fields_autoplaced yes)
@@
 		)
 	)
-	(label "IN2"
+	(label "NTC_Vout(ADC3)"
 		(at 148.59 54.61 0)
 		(fields_autoplaced yes)

Commit message: Made some edits to the main PCB board
Parts:
- added H1, H2, H3, H4: MountingHole, MountingHole:MountingHole_4.3mm_M4, symbol Mechanical:MountingHole

Commit message: finished the PCB board designs
Parts:
- added R6: 20, Resistor_THT:R_Axial_DIN0207_L6.3mm_D2.5mm_P7.62mm_Horizontal, symbol Device:R
- H1, H2, H3, H4: footprint MountingHole:MountingHole_4.3mm_M4 -> MountingHole:MountingHole_3.2mm_M3
Connections:
- net +5V: now also D1.1 (K); no longer J1.2 (Pin_2)
- net OC2B: now also R6.1; no longer J2.2 (Pin_2)
- net at D1.2 (A): now also J1.2 (Pin_2)
- new net: J2.2 (Pin_2), R6.2
- no-connect marks 16 -> 14
Other:
- moved on the sheet: C2, D1
Changed lines of the file:
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@@
 	)
 	(junction
-		(at 49.53 33.02)
-		(diameter 0)
-		(color 0 0 0 0)
-	)
-	(junction
 		(at 233.68 62.23)
 		(diameter 0)
@@
 	)
 	(junction
-		(at 49.53 25.4)
-		(diameter 0)
-		(color 0 0 0 0)
-	)
-	(junction
 		(at 60.96 144.78)
 		(diameter 0)
@@
 	)
 	(junction
+		(at 49.53 25.4)
+		(diameter 0)
+		(color 0 0 0 0)
+	)
+	(junction
 		(at 43.18 132.08)
 		(diameter 0)
@@
 	)
 	(junction
+		(at 49.53 29.21)
+		(diameter 0)
+		(color 0 0 0 0)
+	)
+	(junction
 		(at 68.58 166.37)
 		(diameter 0)
@@
 	)
 	(no_connect
-		(at 34.29 33.02)
-	)
-	(no_connect
 		(at 135.89 80.01)
 	)
@@
 	)
 	(no_connect
-		(at 34.29 25.4)
-	)
-	(no_connect
 		(at 146.05 39.37)
 	)
@@
 	(wire
 		(pts
-			(xy 49.53 33.02) (xy 49.53 40.64)
-		)
-		(stroke
-			(width 0)
-			(type default)
-		)
-	)
-	(wire
-		(pts
 			(xy 238.76 50.8) (xy 241.3 50.8)
 		)
@@
 	(wire
 		(pts
+			(xy 33.02 97.79) (xy 35.56 97.79)
+		)
+		(stroke
+			(width 0)
+			(type default)
+		)
+	)
+	(wire
+		(pts
 			(xy 134.62 165.1) (xy 137.16 165.1)
 		)
@@
 	(wire
 		(pts
+			(xy 43.18 97.79) (xy 50.8 97.79)
+		)
+		(stroke
+			(width 0)
+			(type default)
+		)
+	)
+	(wire
+		(pts
 			(xy 38.1 153.67) (xy 38.1 160.02)
 		)
@@
 	(wire
 		(pts
+			(xy 55.88 36.83) (xy 55.88 38.1)
+		)
+		(stroke
+			(width 0)
+			(type default)
+		)
+	)
+	(wire
+		(pts
 			(xy 116.84 52.07) (xy 120.65 52.07)
 		)
@@
 	(wire
 		(pts
+			(xy 49.53 29.21) (xy 55.88 29.21)
+		)
+		(stroke
+			(width 0)
+			(type default)
+		)
+	)
+	(wire
+		(pts
 			(xy 233.68 62.23) (xy 241.3 62.23)
 		)
@@
 	(wire
 		(pts
-			(xy 49.53 25.4) (xy 49.53 33.02)
-		)
-		(stroke
-			(width 0)
-			(type default)
-		)
-	)
-	(wire
-		(pts
 			(xy 190.5 134.62) (xy 198.12 134.62)
 		)
@@
 	(wire
 		(pts
-			(xy 57.15 33.02) (xy 49.53 33.02)
+			(xy 46.99 60.96) (xy 46.99 64.77)
 		)
 		(stroke
@@
 	(wire
 		(pts
-			(xy 46.99 60.96) (xy 46.99 64.77)
+			(xy 207.01 40.64) (xy 207.01 43.18)
 		)
 		(stroke
@@
 	(wire
 		(pts
-			(xy 207.01 40.64) (xy 207.01 43.18)
+			(xy 49.53 135.89) (xy 43.18 135.89)
 		)
 		(stroke
@@
 	(wire
 		(pts
-			(xy 49.53 135.89) (xy 43.18 135.89)
+			(xy 229.87 68.58) (xy 229.87 74.93)
 		)
 		(stroke
@@
 	(wire
 		(pts
-			(xy 229.87 68.58) (xy 229.87 74.93)
+			(xy 134.62 162.56) (xy 137.16 162.56)
 		)
 		(stroke
@@
 	(wire
 		(pts
-			(xy 134.62 162.56) (xy 137.16 162.56)
+			(xy 128.27 132.08) (xy 139.7 132.08)
 		)
 		(stroke
@@
 	(wire
 		(pts
-			(xy 128.27 132.08) (xy 139.7 132.08)
+			(xy 48.26 100.33) (xy 50.8 100.33)
 		)
 		(stroke
@@
 	(wire
 		(pts
-			(xy 48.26 100.33) (xy 50.8 100.33)
+			(xy 49.53 36.83) (xy 49.53 40.64)
 		)
 		(stroke
@@
 	(wire
 		(pts
-			(xy 233.68 71.12) (xy 241.3 71.12)
+			(xy 49.53 25.4) (xy 49.53 29.21)
 		)
 		(stroke
@@
 	(wire
 		(pts
-			(xy 48.26 97.79) (xy 50.8 97.79)
+			(xy 233.68 71.12) (xy 241.3 71.12)
 		)
 		(stroke
@@
 	)
 	(rectangle
-		(start 34.29 90.17)
+		(start 22.86 88.9)
 		(end 80.01 105.41)
 		(stroke
@@
 	)
 	(label "OC2B"
-		(at 48.26 97.79 180)
+		(at 33.02 97.79 180)
 		(fields_autoplaced yes)
 		(effects
@@
 		)
 	)
+	(netclass_flag ""
+		(length 1)
+		(shape dot)
+		(at 49.53 38.1 270)
+		(fields_autoplaced yes)
+		(effects
+			(font
+				(size 1.27 1.27)
+			)
+			(justify right bottom)
+		)
+		(property "Netclass" "Power"
+			(at 50.53 37.4015 90)
+			(effects
+				(font
+					(size 1.27 1.27)
+					(italic yes)
+				)
+				(justify left)
+				(hide yes)
+			)
+		)
+	)
 	(symbol
 		(lib_id "power:GND")
@@
 	)
 	(symbol
+		(lib_id "Device:R")
+		(at 39.37 97.79 90)
+		(unit 1)
+		(exclude_from_sim no)
+		(in_bom yes)
+		(on_board yes)
+		(dnp no)
+		(fields_autoplaced yes)
+		(property "Reference" "R6"
+			(at 39.37 91.44 90)
+			(effects
+				(font
+					(size 1.27 1.27)
+				)
+			)
+		)
+		(property "Value" "20"
+			(at 39.37 93.98 90)
+			(effects
+				(font
+					(size 1.27 1.27)
+				)
+			)
+		)
+		(property "Footprint" "Resistor_THT:R_Axial_DIN0207_L6.3mm_D2.5mm_P7.62mm_Horizontal"
+			(at 39.37 99.568 90)
+			(effects
+				(font
+					(size 1.27 1.27)
+				)
+				(hide yes)
+			)
+		)
+		(property "Datasheet" "~"
+			(at 39.37 97.79 0)
+			(effects
+				(font
+					(size 1.27 1.27)
+				)
+				(hide yes)
+			)
+		)
+		(property "Description" "Resistor"
+			(at 39.37 97.79 0)
+			(effects
+				(font
+					(size 1.27 1.27)
+				)
+				(hide yes)
+			)
+		)
+		(pin "2"
+		)
+		(pin "1"
+		)
+		(instances
+			(project ""
+				(path "/53da7c59-d564-4ca1-aec6-a8473e4863ca"
+					(reference "R6")
+					(unit 1)
+				)
+			)
+		)
+	)
+	(symbol
 		(lib_id "Connector:Conn_01x03_Pin")
 		(at 246.38 41.91 0)
@@
 			)
 		)
-		(property "Footprint" "MountingHole:MountingHole_4.3mm_M4"
+		(property "Footprint" "MountingHole:MountingHole_3.2mm_M3"
 			(at 100.33 107.95 0)
 			(effects
@@
 			)
 		)
-		(property "Footprint" "MountingHole:MountingHole_4.3mm_M4"
+		(property "Footprint" "MountingHole:MountingHole_3.2mm_M3"
 			(at 100.33 101.6 0)
 			(effects
@@
 	(symbol
 		(lib_id "Device:D_Shockley")
-		(at 34.29 29.21 270)
+		(at 49.53 33.02 270)
 		(unit 1)
 		(exclude_from_sim no)
@@
 		(on_board yes)
 		(dnp no)
-		(fields_autoplaced yes)
 		(property "Reference" "D1"
-			(at 36.83 27.9399 90)
+			(at 36.83 30.734 90)
 			(effects
 				(font
@@
 		)
 		(property "Value" "D_Shockley"
-			(at 36.83 30.4799 90)
+			(at 36.83 33.274 90)
 			(effects
 				(font
@@
 		)
 		(property "Footprint" "Diode_THT:D_DO-41_SOD81_P10.16mm_Horizontal"
-			(at 34.29 29.21 0)
+			(at 49.53 33.02 0)
 			(effects
 				(font
@@
 		)
 		(property "Datasheet" "~"
-			(at 34.29 29.21 0)
+			(at 49.53 33.02 0)
 			(effects
 				(font
@@
 		)
 		(property "Description" "Shockley (PNPN) diode"
-			(at 34.29 29.21 0)
+			(at 49.53 33.02 0)
 			(effects
 				(font
@@
 	(symbol
 		(lib_id "power:GND")
-		(at 57.15 40.64 0)
+		(at 55.88 38.1 0)
 		(unit 1)
 		(exclude_from_sim no)
@@
 		(fields_autoplaced yes)
 		(property "Reference" "#PWR030"
-			(at 57.15 46.99 0)
+			(at 55.88 44.45 0)
 			(effects
 				(font
@@
 		)
 		(property "Value" "GND"
-			(at 57.15 45.72 0)
+			(at 55.88 43.18 0)
 			(effects
 				(font
@@
 		)
 		(property "Footprint" ""
-			(at 57.15 40.64 0)
+			(at 55.88 38.1 0)
 			(effects
 				(font
@@
 		)
 		(property "Datasheet" ""
-			(at 57.15 40.64 0)
+			(at 55.88 38.1 0)
 			(effects
 				(font
@@
 		)
 		(property "Description" "Power symbol creates a global label with name \"GND\" , ground"
-			(at 57.15 40.64 0)
+			(at 55.88 38.1 0)
 			(effects
 				(font
@@
 	(symbol
 		(lib_id "Device:C_Polarized")
-		(at 57.15 36.83 0)
+		(at 55.88 33.02 0)
 		(unit 1)
 		(exclude_from_sim no)
@@
 		(fields_autoplaced yes)
 		(property "Reference" "C2"
-			(at 60.96 34.6709 0)
+			(at 59.69 30.8609 0)
 			(effects
 				(font
@@
 		)
 		(property "Value" "10uF"
-			(at 60.96 37.2109 0)
+			(at 59.69 33.4009 0)
 			(effects
 				(font
@@
 		)
 		(property "Footprint" "Capacitor_THT:CP_Radial_D5.0mm_P2.50mm"
-			(at 58.1152 40.64 0)
+			(at 56.8452 36.83 0)
 			(effects
 				(font
@@
 		)
 		(property "Datasheet" "~"
-			(at 57.15 36.83 0)
+			(at 55.88 33.02 0)
 			(effects
 				(font
@@
 		)
 		(property "Description" "Polarized capacitor"
-			(at 57.15 36.83 0)
+			(at 55.88 33.02 0)
 			(effects
 				(font
@@
 			)
 		)
-		(property "Footprint" "MountingHole:MountingHole_4.3mm_M4"
+		(property "Footprint" "MountingHole:MountingHole_3.2mm_M3"
 			(at 90.17 101.6 0)
 			(effects
@@
 			)
 		)
-		(property "Footprint" "MountingHole:MountingHole_4.3mm_M4"
+		(property "Footprint" "MountingHole:MountingHole_3.2mm_M3"
 			(at 90.17 107.95 0)
 			(effects
