File: Main PCB/Main PCB.kicad_sch (KiCad schematic)
At the start: 43 parts, among them J1 Power Input, J10 Conn_01x03_Pin, J11 Conn_01x03_Pin, J12 Conn_01x03_Pin, J13 Conn_01x03_Pin, J14 Conn_01x03_Pin, J15 Conn_01x03_Pin, J16 Spare I2C PINS, J2 2nd PCB, J3 Servo Motor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

Commit message: Second revision
Parts:
- removed C1: 0.1uF, Capacitor_THT:CP_Radial_D5.0mm_P2.50mm, symbol Device:C_Polarized
- removed C4: 33uF, Capacitor_THT:C_Disc_D3.8mm_W2.6mm_P2.50mm, symbol Device:C
- removed J7: GPS Module, Connector_PinSocket_2.54mm:PinSocket_1x04_P2.54mm_Vertical, symbol Connector:Conn_01x04_Socket
- removed U1: TLV9002, Package_DIP:DIP-8_W7.62mm, symbol Simulation_SPICE:OPAMP
- added C1, C12: 10nF, Capacitor_THT:C_Disc_D3.8mm_W2.6mm_P2.50mm, symbol Device:C
- added C13: 10uF, Capacitor_THT:C_Disc_D5.0mm_W2.5mm_P5.00mm, symbol Device:C
- added J17: Trigger Pin (backup), Connector_PinHeader_2.54mm:PinHeader_1x01_P2.54mm_Vertical, symbol Connector:Conn_01x01_Pin
- added J7: Conn_01x05_Pin, Connector_PinHeader_2.54mm:PinHeader_1x05_P2.54mm_Vertical, symbol Connector:Conn_01x05_Pin
- added R7: 100, Resistor_THT:R_Axial_DIN0207_L6.3mm_D2.5mm_P10.16mm_Horizontal, symbol Device:R
- added U1: CA3140, Package_DIP:DIP-8_W7.62mm, symbol Amplifier_Operational:CA3140
- C3: value 0.1uF -> 1uF
- R1: value 10.8k -> 11k
- R2: value 3.01k -> 3k
- R3: value 3.09k -> 3k
Connections:
- net +5V: now also C1.2, C12.1, R7.1, U1.7 (V+); no longer R2.1
- net GND: now also U2.6 (INH), C1.1, C12.2, U1.4 (V-)
- net NTC_Vout(ADC3): now also C13.1, U1.6
- net at R1.1, TH1.1: now also U1.3 (+)
- net at R2.2, R3.1, R5.2: now also C13.2, U1.2 (-)
- net D1/TX: now reaches A1.1 (D1/TX)
- net D1/TX: now also J7.1 (Pin_1)
- net Trigger: now reaches A1.10 (D7)
- net Trigger: now also J17.1 (Pin_1)
- net D0/RX: now reaches A1.2 (D0/RX)
- net D0/RX: now also J7.2 (Pin_2)
- net PC6/RESET: now reaches A1.3 (~{RESET})
- net PC6/RESET: now also J7.3 (Pin_3)
- net D2: now reaches A1.5 (D2)
- net D2: now also J7.4 (Pin_4)
- net D4: now reaches A1.7 (D4)
- net D4: now also J7.5 (Pin_5)
- new net: R2.1, R7.2
- no-connect marks 14 -> 10
Other:
- moved on the sheet: C11, C3, C7, C9, J16, J6, R5

Commit message: Added manual vias
Connections:
- net GND: now also A1.29 (GND)
- no-connect marks 10 -> 9
Other:
- moved on the sheet: C5
Changed lines of the file:
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@@
 	)
 	(junction
+		(at 133.35 80.01)
+		(diameter 0)
+		(color 0 0 0 0)
+	)
+	(junction
 		(at 85.09 157.48)
 		(diameter 0)
@@
 	)
 	(junction
+		(at 130.81 25.4)
+		(diameter 0)
+		(color 0 0 0 0)
+	)
+	(junction
 		(at 83.82 170.18)
 		(diameter 0)
@@
 	)
 	(junction
-		(at 130.81 26.67)
-		(diameter 0)
-		(color 0 0 0 0)
-	)
-	(junction
 		(at 38.1 160.02)
 		(diameter 0)
@@
 	)
 	(no_connect
-		(at 138.43 29.21)
-	)
-	(no_connect
 		(at 71.12 149.86)
 	)
@@
 	)
 	(no_connect
-		(at 135.89 80.01)
+		(at 138.43 29.21)
 	)
 	(no_connect
@@
 	(wire
 		(pts
-			(xy 130.81 26.67) (xy 130.81 29.21)
-		)
-		(stroke
-			(width 0)
-			(type default)
-		)
-	)
-	(wire
-		(pts
 			(xy 139.7 129.54) (xy 151.13 129.54)
 		)
@@
 	(wire
 		(pts
+			(xy 133.35 80.01) (xy 135.89 80.01)
+		)
+		(stroke
+			(width 0)
+			(type default)
+		)
+	)
+	(wire
+		(pts
 			(xy 43.18 97.79) (xy 50.8 97.79)
 		)
@@
 	(wire
 		(pts
-			(xy 130.81 24.13) (xy 130.81 26.67)
+			(xy 130.81 22.86) (xy 130.81 25.4)
 		)
 		(stroke
@@
 	(wire
 		(pts
+			(xy 130.81 25.4) (xy 130.81 29.21)
+		)
+		(stroke
+			(width 0)
+			(type default)
+		)
+	)
+	(wire
+		(pts
 			(xy 85.09 144.78) (xy 85.09 157.48)
 		)
@@
 	(symbol
 		(lib_id "power:GND")
-		(at 123.19 26.67 270)
+		(at 123.19 25.4 270)
 		(unit 1)
 		(exclude_from_sim no)
@@
 		(fields_autoplaced yes)
 		(property "Reference" "#PWR025"
-			(at 116.84 26.67 0)
+			(at 116.84 25.4 0)
 			(effects
 				(font
@@
 		)
 		(property "Value" "GND"
-			(at 119.38 26.6699 90)
+			(at 119.38 25.3999 90)
 			(effects
 				(font
@@
 		)
 		(property "Footprint" ""
-			(at 123.19 26.67 0)
+			(at 123.19 25.4 0)
 			(effects
 				(font
@@
 		)
 		(property "Datasheet" ""
-			(at 123.19 26.67 0)
+			(at 123.19 25.4 0)
 			(effects
 				(font
@@
 		)
 		(property "Description" "Power symbol creates a global label with name \"GND\" , ground"
-			(at 123.19 26.67 0)
+			(at 123.19 25.4 0)
 			(effects
 				(font
@@
 	(symbol
 		(lib_id "Device:C_Polarized")
-		(at 127 26.67 270)
+		(at 127 25.4 270)
 		(unit 1)
 		(exclude_from_sim no)
@@
 		(dnp no)
 		(property "Reference" "C5"
-			(at 123.952 19.812 90)
+			(at 123.952 18.542 90)
 			(effects
 				(font
@@
 		)
 		(property "Value" "0.1uF"
-			(at 123.444 22.098 90)
+			(at 123.444 20.828 90)
 			(effects
 				(font
@@
 		)
 		(property "Footprint" "Capacitor_THT:CP_Radial_D5.0mm_P2.50mm"
-			(at 123.19 27.6352 0)
+			(at 123.19 26.3652 0)
 			(effects
 				(font
@@
 		)
 		(property "Datasheet" "~"
-			(at 127 26.67 0)
+			(at 127 25.4 0)
 			(effects
 				(font
@@
 		)
 		(property "Description" "Polarized capacitor"
-			(at 127 26.67 0)
+			(at 127 25.4 0)
 			(effects
 				(font
@@
 		)
 		(property "Sim.Device" ""
-			(at 127 26.67 0)
+			(at 127 25.4 0)
 			(effects
 				(font
@@
 		)
 		(property "Sim.Library" ""
-			(at 127 26.67 0)
+			(at 127 25.4 0)
 			(effects
 				(font
@@
 		)
 		(property "Sim.Name" ""
-			(at 127 26.67 0)
+			(at 127 25.4 0)
 			(effects
 				(font
@@
 		)
 		(property "Sim.Pins" ""
-			(at 127 26.67 0)
+			(at 127 25.4 0)
 			(effects
 				(font
@@
 	(symbol
 		(lib_id "power:+5V")
-		(at 130.81 24.13 0)
+		(at 130.81 22.86 0)
 		(unit 1)
 		(exclude_from_sim no)
@@
 		(fields_autoplaced yes)
 		(property "Reference" "#PWR02"
-			(at 130.81 27.94 0)
+			(at 130.81 26.67 0)
 			(effects
 				(font
@@
 		)
 		(property "Value" "+5V"
-			(at 130.81 19.05 0)
+			(at 130.81 17.78 0)
 			(effects
 				(font
@@
 		)
 		(property "Footprint" ""
-			(at 130.81 24.13 0)
+			(at 130.81 22.86 0)
 			(effects
 				(font
@@
 		)
 		(property "Datasheet" ""
-			(at 130.81 24.13 0)
+			(at 130.81 22.86 0)
 			(effects
 				(font
@@
 		)
 		(property "Description" "Power symbol creates a global label with name \"+5V\""
-			(at 130.81 24.13 0)
+			(at 130.81 22.86 0)
 			(effects
 				(font
